File: Main Project Logic Board/ss_main_logic/ss_main_logic.kicad_pcb (KiCad board)
At the start: 4 copper layers, 60 x 50 mm, 17 parts, among them J1 Conn_01x06_Pin, J2 KeyPAD, J3 Conn_01x03_Pin, J4 Conn_01x03_Pin, J5 Screw_Terminal_01x02, J6 Conn_01x03_Pin, U1 PIC24FJ128GA010-I_PT, U2 RN4870-V_RM118

Commit message: Added different BLE and LEDs
Parts:
- removed U2: RN4870-V_RM118, footprints:RN4870_MCH
- added D1: R_LED, LED_SMD:LED_0603_1608Metric, F.Cu at (102.0, 127.2)
- added D2: R_LED, LED_SMD:LED_0603_1608Metric, F.Cu at (131.2, 129.5)
- added D3: R_LED, LED_SMD:LED_0603_1608Metric, F.Cu at (131.2, 132.1)
- added D4: R_LED, LED_SMD:LED_0603_1608Metric, F.Cu at (131.2, 134.7)
- added D5: R_LED, LED_SMD:LED_0603_1608Metric, F.Cu at (131.2, 137.3)
- added J7: Conn_01x08_Socket, Connector_PinSocket_2.54mm:PinSocket_1x08_P2.54mm_Vertical, F.Cu at (99.1, 92.0)
- added J8: Conn_01x08_Socket, Connector_PinSocket_2.54mm:PinSocket_1x08_P2.54mm_Vertical, F.Cu at (122.0, 92.0)
- added J9: Conn_01x02_Pin, Connector_PinHeader_2.54mm:PinHeader_1x02_P2.54mm_Vertical, F.Cu at (167.5, 126.5)
- added R3: 65, Resistor_SMD:R_1210_3225Metric, F.Cu at (102.0, 121.5)
- added R4: 65, Resistor_SMD:R_1210_3225Metric, F.Cu at (138.0, 126.0)
- added R5: 65, Resistor_SMD:R_1210_3225Metric, F.Cu at (138.0, 129.5)
- added R6: 65, Resistor_SMD:R_1210_3225Metric, F.Cu at (138.0, 133.0)
- added R7: 65, Resistor_SMD:R_1210_3225Metric, F.Cu at (138.0, 136.5)
- moved C4 1.00 mm to (147.0, 126.0)
Connections:
- U1 pad 26: unconnected-(U1-PGC2/EMUC2/AN6/OCFA/RB6-Pad26) -> Net-(U1-PGC2/EMUC2/AN6/OCFA/RB6)
- U1 pad 27: unconnected-(U1-PGD2/EMUD2/AN7/RB7-Pad27) -> Net-(U1-PGD2/EMUD2/AN7/RB7)
- U1 pad 28: unconnected-(U1-PMA7/VREF-/RA9-Pad28) -> Net-(U1-PMA7/VREF-/RA9)
- U1 pad 29: unconnected-(U1-PMA6/VREF+/RA10-Pad29) -> Net-(U1-PMA6/VREF+/RA10)
- U1 pad 49: unconnected-(U1-PMA9/U2RX/CN17/RF4-Pad49) -> /U2RX
- U1 pad 50: unconnected-(U1-PMA8/U2TX/CN18/RF5-Pad50) -> /U2TX
Routing:
- net Net-(U1-PMA6/VREF+/RA10): track 0.00 -> 17.7 mm
- net /U2RX: track 0.00 -> 14.5 mm, vias 0 -> 1
- net Net-(U1-PMA7/VREF-/RA9): track 0.00 -> 14.0 mm
- net /U2TX: track 0.00 -> 12.5 mm, vias 0 -> 1
- net Net-(U1-PGD2/EMUD2/AN7/RB7): track 0.00 -> 10.3 mm
- net Net-(U1-PGC2/EMUC2/AN6/OCFA/RB6): track 0.00 -> 7.30 mm
- net GND: track 53.7 -> 46.5 mm, vias 13 -> 14
- net /BLE_UART_RX: track 42.8 -> 49.9 mm, vias 2 -> 1
- net /BLE_UART_TX: track 39.7 -> 46.6 mm, vias 2 -> 1
- net Net-(D2-A): track 0.00 -> 6.02 mm
- net Net-(D3-A): track 0.00 -> 5.65 mm
- net Net-(D4-A): track 0.00 -> 5.27 mm
- net Net-(D5-A): track 0.00 -> 4.89 mm
- net Net-(D1-A): track 0.00 -> 3.42 mm
- net +3.3V: track 24.8 -> 21.4 mm
Other:
- board size 60 x 50 mm -> 73.5 x 50 mm
- board text added: "+"
- board text added: "-"
- board text added: "3V3"
- board text added: "GND"
- board text added: "L-DIR"
- board text added: "L-SLP"
- board text added: "L-STP"
- board text added: "MCLR"
- board text added: "PCK"
- board text added: "PGD"
- board text added: "W-Dir"
- board text added: "W-SLP"
- board text removed: "L-STEP"

Commit message: Added some gerbers
Other:
- board text added: "3V3 I"
Changed lines of the file:
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@@
+		)
+	)
+	(gr_text "3V3 I"
+		(at 97 130 0)
+		(layer "F.SilkS")
+		(effects
+			(font
+				(size 1 1)
+				(thickness 0.2)
+				(bold yes)
+			)
+			(justify left bottom)
 		)
 	)
